File: Project (PCB)/Eagle Files/CoffeeHeater.sch (EAGLE design)
At the start: 40 parts, among them Q1 BSS138, U1 POCKETBEAGLE, U2 0.56_HEX_BACKPACK, U3 TPS63060

Commit message: Updated connections
Parts:
- renumbered U$3 to D2
Connections:
- net I2C_SCL: no longer R3.1
- net I2C_SDA: now also R3.1
Changed lines of the file:
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@@
 <part name="GND3" library="ENGI301" deviceset="GND" device=""/>
 <part name="SUPPLY7" library="ENGI301" deviceset="VDD_5V" device=""/>
-<part name="U$3" library="CoffeeHeater" deviceset="DIODE" device=""/>
+<part name="D2" library="CoffeeHeater" deviceset="DIODE" device=""/>
 <part name="U$4" library="CoffeeHeater" deviceset="HEATING_PAD" device=""/>
 <part name="GND4" library="ENGI301" deviceset="GND" device=""/>
@@
 <attribute name="VALUE" x="187.96" y="176.784" size="1.778" layer="96" align="center"/>
 </instance>
-<instance part="U$3" gate="G$1" x="323.215" y="144.145"/>
+<instance part="D2" gate="G$1" x="323.215" y="144.145"/>
 <instance part="U$4" gate="G$1" x="345.44" y="124.46" rot="R270">
 <attribute name="NAME" x="347.98" y="127" size="1.778" layer="95" rot="R270" display="off"/>
@@
 <segment>
 <pinref part="U2" gate="G$1" pin="SDA"/>
-<wire x1="205.74" y1="213.36" x2="154.94" y2="213.36" width="0.1524" layer="91"/>
+<wire x1="205.74" y1="213.36" x2="175.26" y2="213.36" width="0.1524" layer="91"/>
 <label x="152.4" y="213.36" size="1.778" layer="95"/>
+<pinref part="R3" gate="G$1" pin="1"/>
+<wire x1="175.26" y1="213.36" x2="154.94" y2="213.36" width="0.1524" layer="91"/>
+<wire x1="175.26" y1="223.52" x2="175.26" y2="213.36" width="0.1524" layer="91"/>
+<junction x="175.26" y="213.36"/>
 </segment>
 <segment>
@@
 <segment>
 <pinref part="U2" gate="G$1" pin="SCL"/>
-<wire x1="205.74" y1="218.44" x2="175.26" y2="218.44" width="0.1524" layer="91"/>
+<wire x1="205.74" y1="218.44" x2="165.1" y2="218.44" width="0.1524" layer="91"/>
 <pinref part="R2" gate="G$1" pin="1"/>
-<wire x1="175.26" y1="218.44" x2="165.1" y2="218.44" width="0.1524" layer="91"/>
 <wire x1="165.1" y1="218.44" x2="154.94" y2="218.44" width="0.1524" layer="91"/>
 <wire x1="165.1" y1="223.52" x2="165.1" y2="218.44" width="0.1524" layer="91"/>
 <junction x="165.1" y="218.44"/>
-<pinref part="R3" gate="G$1" pin="1"/>
-<wire x1="175.26" y1="223.52" x2="175.26" y2="218.44" width="0.1524" layer="91"/>
-<junction x="175.26" y="218.44"/>
 <label x="152.4" y="218.44" size="1.778" layer="95"/>
 </segment>
@@
 <net name="BASE" class="0">
 <segment>
-<pinref part="U$3" gate="G$1" pin="OUT"/>
+<pinref part="D2" gate="G$1" pin="OUT"/>
 <pinref part="U$2" gate="G$1" pin="B"/>
 <wire x1="332.105" y1="144.145" x2="335.28" y2="144.145" width="0.1524" layer="91"/>
@@
 <net name="HEAT_CONTROL" class="0">
 <segment>
-<pinref part="U$3" gate="G$1" pin="IN"/>
+<pinref part="D2" gate="G$1" pin="IN"/>
 <wire x1="318.135" y1="144.145" x2="300.355" y2="144.145" width="0.1524" layer="91"/>
 <label x="299.72" y="144.78" size="1.778" layer="95"/>

Commit message: Updated library and created BOM
Parts:
- renumbered U$1 to T1, U$2 to TR1, U$4 to H1
Changed lines of the file:
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@@
 <part name="GND10" library="ENGI301" deviceset="GND" device=""/>
 <part name="GND11" library="ENGI301" deviceset="GND" device=""/>
-<part name="U$1" library="CoffeeHeater" deviceset="DS18B20_TEMP_SENSOR" device=""/>
-<part name="U$2" library="CoffeeHeater" deviceset="TIP32C_TRANSISTOR" device=""/>
+<part name="T1" library="CoffeeHeater" deviceset="DS18B20_TEMP_SENSOR" device=""/>
+<part name="TR1" library="CoffeeHeater" deviceset="TIP32C_TRANSISTOR" device=""/>
 <part name="GND3" library="ENGI301" deviceset="GND" device=""/>
 <part name="SUPPLY7" library="ENGI301" deviceset="VDD_5V" device=""/>
 <part name="D2" library="CoffeeHeater" deviceset="DIODE" device=""/>
-<part name="U$4" library="CoffeeHeater" deviceset="HEATING_PAD" device=""/>
+<part name="H1" library="CoffeeHeater" deviceset="HEATING_PAD" device=""/>
 <part name="GND4" library="ENGI301" deviceset="GND" device=""/>
 <part name="R4" library="ENGI301" deviceset="R_" device="R0603" value="2.2k"/>
@@
 <attribute name="VALUE" x="271.78" y="124.46" size="1.778" layer="96" rot="R90"/>
 </instance>
-<instance part="U$1" gate="G$1" x="160.02" y="137.16"/>
-<instance part="U$2" gate="G$1" x="340.36" y="144.145"/>
+<instance part="T1" gate="G$1" x="160.02" y="137.16"/>
+<instance part="TR1" gate="G$1" x="340.36" y="144.145"/>
 <instance part="GND3" gate="1" x="163.83" y="170.18" rot="R180">
 <attribute name="VALUE" x="166.37" y="172.72" size="1.778" layer="96" rot="R180"/>
@@
 </instance>
 <instance part="D2" gate="G$1" x="323.215" y="144.145"/>
-<instance part="U$4" gate="G$1" x="345.44" y="124.46" rot="R270">
+<instance part="H1" gate="G$1" x="345.44" y="124.46" rot="R270">
 <attribute name="NAME" x="347.98" y="127" size="1.778" layer="95" rot="R270" display="off"/>
 <attribute name="VALUE" x="347.98" y="129.54" size="1.778" layer="96" rot="R270"/>
@@
 <pinref part="SUPPLY7" gate="G$1" pin="VDD_5V"/>
 <wire x1="187.96" y1="167.64" x2="187.96" y2="170.18" width="0.1524" layer="91"/>
-<pinref part="U$1" gate="G$1" pin="VDD"/>
+<pinref part="T1" gate="G$1" pin="VDD"/>
 <wire x1="171.45" y1="160.02" x2="187.96" y2="160.02" width="0.1524" layer="91"/>
 <wire x1="187.96" y1="160.02" x2="187.96" y2="167.64" width="0.1524" layer="91"/>
@@
 <segment>
 <pinref part="GND3" gate="1" pin="GND"/>
-<pinref part="U$1" gate="G$1" pin="GND"/>
+<pinref part="T1" gate="G$1" pin="GND"/>
 <wire x1="163.83" y1="167.64" x2="163.83" y2="160.02" width="0.1524" layer="91"/>
 </segment>
@@
 </segment>
 <segment>
-<pinref part="U$4" gate="G$1" pin="2"/>
+<pinref part="H1" gate="G$1" pin="2"/>
 <pinref part="GND4" gate="1" pin="GND"/>
 <wire x1="345.44" y1="119.38" x2="345.44" y2="111.76" width="0.1524" layer="91"/>
@@
 <segment>
 <pinref part="D2" gate="G$1" pin="OUT"/>
-<pinref part="U$2" gate="G$1" pin="B"/>
+<pinref part="TR1" gate="G$1" pin="B"/>
 <wire x1="332.105" y1="144.145" x2="335.28" y2="144.145" width="0.1524" layer="91"/>
 </segment>
@@
 <net name="TEMP" class="0">
 <segment>
-<pinref part="U$1" gate="G$1" pin="DQ"/>
+<pinref part="T1" gate="G$1" pin="DQ"/>
 <wire x1="167.64" y1="160.02" x2="167.64" y2="167.64" width="0.1524" layer="91"/>
 <label x="167.64" y="160.02" size="1.778" layer="95" rot="R90"/>
@@
 </segment>
 <segment>
-<pinref part="U$2" gate="G$1" pin="C"/>
+<pinref part="TR1" gate="G$1" pin="C"/>
 <wire x1="345.44" y1="154.305" x2="345.44" y2="163.83" width="0.1524" layer="91"/>
 <label x="344.17" y="156.21" size="1.778" layer="95" rot="R90"/>
@@
 <net name="N$1" class="0">
 <segment>
-<pinref part="U$2" gate="G$1" pin="E"/>
-<pinref part="U$4" gate="G$1" pin="1"/>
+<pinref part="TR1" gate="G$1" pin="E"/>
+<pinref part="H1" gate="G$1" pin="1"/>
 <wire x1="345.44" y1="133.985" x2="345.44" y2="129.54" width="0.1524" layer="91"/>
 </segment>
